File: NeoWall.kicad_pcb (KiCad board)
At the start: 2 copper layers, 70 x 70 mm, 15 parts, among them P1 CONN_01X03, P2 CONN_01X03, P3 CONN_01X03, P4 CONN_01X03

Commit message: Optimize cap positions
Parts:
- turned C4 to 180 degrees
